File: PCB files/MainPCB/MainPCB.kicad_sch (KiCad schematic)
At the start: 123 parts, among them IC1 CYPD3177-24LQXQ, P1 Solder_Pad, P15 Solder_Pad, P16 Solder_Pad, P18 Solder_Pad, P19 Solder_Pad, P20 Solder_Pad, P21 Solder_Pad, P22 Solder_Pad, P25 Solder_Pad, P26 Solder_Pad, P27 Solder_Pad, P28 Solder_Pad, P29 Solder_Pad, P3 Solder_Pad, P30 Solder_Pad, P31 Solder_Pad, P32 Solder_Pad, P33 Solder_Pad, P34 Solder_Pad, P35 Solder_Pad, P4 Solder_Pad, P5 Solder_Pad, SW1 TS-1185EC-C-D-B, SW2 TS-1185EC-C-D-B, SW3 SK-3245S-L3-B, SW4 TS-1185EC-C-D-B, U1 SN74LVC1G373DBVR, U1 TPS53319DQPR, U1 TPS62933DRLR, U10 MSM261D4030H1CPM, U12 AO3400A, U14 SN74LVC2T45DCUR, U15 74LVC2G04DW-7, U16 X6511WR-03H-C30D60-R2, U17 X6511WR-03H-C30D60-R2, U18 X6511WR-03H-C30D60-R2, U19 X6511WR-03H-C30D60-R2, U2 TYPE-C-31-M-22, U21 X6511WR-06H-C30D60-R2, U22 X6511WR-06H-C30D60-R2, U23 ESP32-S3-WROOM-1-N8, U24 SN74LVC2T45DCUR, U4 AP40P05, U5 MDA1050-2R2M, U6 HSM4805, U8 AP40P05

Commit message: started redesign of pcb and added test for atopile
Parts:
- removed C1, C2, C30, C35, C37: 0.1uF, Capacitor_SMD:C_0402_1005Metric, symbol Device:C
- removed C11 (x2): 1nF, Capacitor_SMD:C_0402_1005Metric, symbol Device:C
- removed C12, C13, C14: 22uF X5R, Capacitor_SMD:C_1206_3216Metric, symbol Device:C
- removed C14 (x3): 47uF, Capacitor_SMD:C_1206_3216Metric, symbol Device:C
- removed C15: 4.7uF, Capacitor_SMD:C_1206_3216Metric, symbol Device:C
- removed C16, C17: 1uF, Capacitor_SMD:C_0603_1608Metric, symbol Device:C
- removed C3: 33nF, Capacitor_SMD:C_0603_1608Metric, symbol Device:C
- removed C4: 10uF, Capacitor_SMD:C_0805_2012Metric, symbol Device:C
- removed C5: 47pF, Capacitor_SMD:C_0402_1005Metric, symbol Device:C
- removed C6: 47uF, Capacitor_SMD:C_0805_2012Metric, symbol Device:C
- removed D2: WS2812B, LED_SMD:LED_WS2812B_PLCC4_5.0x5.0mm_P3.2mm, symbol LED:WS2812B
- removed L1: CPY201209T-4R7M-NP, footprint:L0805, symbol MyParts:CPY201209T-4R7M-NP
- removed R1: 30.9K, Resistor_SMD:R_0402_1005Metric, symbol Device:R
- removed R11: 1K, Resistor_SMD:R_0603_1608Metric, symbol Device:R
- removed R15, R2: 105K, Resistor_SMD:R_0603_1608Metric, symbol Device:R
- removed R15, R19, R21: 100K, Resistor_SMD:R_0603_1608Metric, symbol Device:10K 0603
- removed R2: 10K, Resistor_SMD:R_0402_1005Metric, symbol Device:R
- removed R2: 51K, Resistor_SMD:R_0603_1608Metric, symbol Device:R
- removed R2: 220K, Resistor_SMD:R_0603_1608Metric, symbol Device:R
- removed R25 (x2): 5.1K, Resistor_SMD:R_0402_1005Metric, symbol Device:R
- removed R25: 2.4K, Resistor_SMD:R_0402_1005Metric, symbol Device:R
- removed R28: 100K, Resistor_SMD:R_0603_1608Metric, symbol Device:R
- removed R3: 71.5K, Resistor_SMD:R_0603_1608Metric_Pad0.98x0.95mm_HandSolder, symbol Device:R
- removed R3: 150K, Resistor_SMD:R_0603_1608Metric, symbol Device:R
- removed R3: 1.8K, Resistor_SMD:R_0603_1608Metric, symbol Device:R
- removed R3: 10K, Resistor_SMD:R_0603_1608Metric_Pad0.98x0.95mm_HandSolder, symbol Device:R
- removed R30: 5.1K, Resistor_SMD:R_0603_1608Metric, symbol Device:5.1K 1% 0603
- removed SW1: TS-1185EC-C-D-B, footprint:SW-SMD_4P-L3.7-W3.0-P1.50-LS4.7, symbol MyParts:TS-1185EC-C-D-B
- removed SW3: SK-3245S-L3-B, footprint:SW-SMD_SK-3245S-L3-B, symbol MyParts:SK-3245S-L3-B
- removed U1: TPS62933DRLR, footprint:SOT-583-8_L2.1-W1.2-P0.50-LS1.6-BR, symbol MyParts:TPS62933DRLR
- removed U1: TPS53319DQPR, footprint:LSON-CLIP-22_L6.0-W5.0-P0.50-BL-EP, symbol MyParts:TPS53319DQPR
- removed U1: SN74LVC1G373DBVR, footprint:SOT-23-6_L2.9-W1.6-P0.95-LS2.8-BR, symbol MyParts:SN74LVC1G373DBVR
- removed U12: AO3400A, footprint:SOT-23-3_L2.9-W1.6-P1.90-LS2.8-BR, symbol MyParts:AO3400A
- removed U16, U17, U18, U19: X6511WR-03H-C30D60-R2, footprint:HDR-TH_3P-P2.54-H-M-W10.4, symbol MyParts:X6511WR-03H-C30D60-R2
- removed U21, U22: X6511WR-06H-C30D60-R2, footprint:HDR-TH_6P-P2.54-H-M-W10.4, symbol MyParts:X6511WR-06H-C30D60-R2
- removed U23: ESP32-S3-WROOM-1-N8, Espressif:ESP32-S3-WROOM-1, symbol Espressif:ESP32-S3-WROOM-1
- removed U4, U8: AP40P05, footprint:SOT-23-3_L2.9-W1.3-P1.90-LS2.4-BR, symbol MyParts:AP40P05
- removed U5: MDA1050-2R2M, footprint:IND-SMD_L11.5-W10.0_MCF-1050, symbol MyParts:MS1040-R68M
- added C22, C8, C9: 0.1uF, Capacitor_SMD:C_0402_1005Metric, symbol Device:C
- added C24: 10uF, Capacitor_SMD:C_0603_1608Metric, symbol Device:10uF 0603
- added J1, J2, J3, J4: Conn_01x03_Pin, Connector_PinHeader_2.54mm:PinHeader_1x03_P2.54mm_Vertical, symbol Connector:Conn_01x03_Pin
- added J5, J6: Conn_01x02_Pin, Connector_PinHeader_2.54mm:PinHeader_1x02_P2.54mm_Vertical, symbol Connector:Conn_01x02_Pin
- added Q1: CSD16301Q2, Package_SON:Texas_DQK, symbol Transistor_FET:CSD16301Q2
- added R22, R8: 5.1K, Resistor_SMD:R_0402_1005Metric, symbol Device:5.1K 1% 0603
- added R23: 1K, Resistor_SMD:R_0402_1005Metric, symbol Device:5.1K 1% 0603
- added R6: 20K, Resistor_SMD:R_0402_1005Metric, symbol Device:5.1K 1% 0603
- added U1: TPS40305DRCR, footprint:VSON-10_L3.0-W3.0-P0.50-BL-EP_TPS62410DRCR, symbol MyParts:TPS40305DRCR
- added U11: SN74LVC2T45DCUR, footprint:VSSOP-8_L2.4-W2.1-P0.50-LS3.2-BR, symbol MyParts:SN74LVC2T45DCUR
- added U17: ESP32-WROOM-32E-N8R2, Espressif:ESP32-WROOM-32E, symbol MyParts:ESP32-WROOM-32E
- added U22: UMH3N, footprint:SC-70-6_L2.2-W1.3-P0.65-LS2.1-BR, symbol LCSC:UMH3N
- added U25: CP2102N-A02-GQFN24R, footprint:QFN-24_L4.0-W4.0-P0.50-TL-EP2.6, symbol MyParts:CP2102N-A02-GQFN24R
- added U28: SP0503BAHTG, footprint:SOT-143-4_L2.9-W1.3-P1.92-LS2.4-BL, symbol MyParts:SP0503BAHTG_C3040626
- added U3: CSD17581Q3AT, footprint:PDFN-8_L3.2-W3.0-P0.65-LS3.3-BL-1, symbol MyParts:CSD17581Q3AT
- added U4: TMPC1206HP-1R5MG-D, footprint:IND-SMD_L13.5-W12.6_TMPC1206HP-1R5MG-D, symbol MyParts:TMPC1206HP-1R5MG-D
- added U6: APM4953_C7473297, footprint:SOP-8_L4.9-W3.9-P1.27-LS6.0-BL, symbol MyParts:APM4953_C7473297
- added U9: AMS1117-3_3, footprint:SOT-223-3_L6.5-W3.4-P2.30-LS7.0-BR, symbol MyParts:AMS1117-3_3
- R10: value 5.1K -> 62; LCSC # C25905 -> C4962
Connections:
- net IO6/USB PD AMPS DETECTION is gone; now on net GND: IC1.5 (ISNK_COARSE)
- net USB_PD_IC_VBUS_MIN is gone; now on net GND: IC1.1 (VBUS_MIN)
- net +3.3V: now also C22.1, C24.1, C9.2, R22.1, R23.2, U11.8 (VCCB), U17.2 (3V3), U25.5 (VIO), U25.6 (VDD), U25.7 (VREGIN)
- net +5V: now also U4.2, U9.3 (VIN); no longer C21.2, C28.2, P1.1, P1.1, U14.1 (VCCA), U24.1 (VCCA)
- net ACTIONBUTTON_EXTERNAL: now also J5.2 (Pin_2), U17.25 (IO0)
- net EN: now also U22.6 (C); no longer C25.2, SW4.2
- net GND: now also C22.2, C24.2, C8.1, C9.1, J1.3 (Pin_3), J2.3 (Pin_3), J3.3 (Pin_3), J4.3 (Pin_3), J5.1 (Pin_1), R8.1, U11.4 (GND), U11.5 (DIR), U17.1 (GND), U17.15 (GND), U17.38 (GND), U17.39 (GND), U25.2 (GND), U25.25 (GND), U28.1; no longer R10.1
- net IO12/I2S WS: no longer U10.2 (L/R)
- net IO13/I2S SCK: no longer U10.3 (CLK)
- net IO14/I2S SD: no longer U10.4 (DATA)
- net IO19/USB D-: no longer U2.5 (DN2), U2.7 (DN1)
- net IO1/POWERBUTTON: no longer U15.6 (1Y)
- net IO20/USB D+: no longer U2.6 (DP1), U2.8 (DP2)
- net IO3/ACTIONBUTTON: no longer U15.4 (2Y)
- net RXD0: now also U17.34 (RXD0), U25.21 (TXD)
- net TXD0: now also U17.35 (TXD0), U25.20 (RXD)
- net USB_PD_IC_VDC_OUT: now also R6.2
- net ACTIONBUTTON LED RING DATA OUT: now reaches R10.2
- net IO41/LED2 renamed IO17/LED STRIP 2
- net IO17/LED STRIP 2: now also U17.28 (IO17)
- net IO42/LED1 renamed IO16/LED STRIP 1
- net IO16/LED STRIP 1: now also U17.27 (IO16)
- net IO4/LED3 renamed IO18/LED STRIP 3
- net IO18/LED STRIP 3: now also U17.30 (IO18)
- net IO5/LED4 renamed IO19/LED STRIP 4
- net IO19/LED STRIP 4: now also U17.31 (IO19)
- net LED1 DATA OUT renamed LED STRIP 1 DATA OUT
- net LED STRIP 1 DATA OUT: now also J1.2 (Pin_2)
- net LED2 DATA OUT renamed LED STRIP 2 DATA OUT
- net LED STRIP 2 DATA OUT: now also J2.2 (Pin_2)
- net LED3 DATA OUT renamed LED STRIP 3 DATA OUT
- net LED STRIP 3 DATA OUT: now also J3.2 (Pin_2)
- net LED4 DATA OUT renamed LED STRIP 4 DATA OUT
- net LED STRIP 4 DATA OUT: now also J4.2 (Pin_2)
- net POWERBUTTON_EXTERNAL: no longer names the net of U15.1 (1A)
- new net: R10.1, U11.2 (A1)
- new net: R6.1, R8.2, U25.8 (VBUS)
- new net: R23.1, U25.9 (RSTb)
- new net: U17.17 (NC), U17.18 (NC), U17.19 (NC), U17.20 (NC), U17.21 (NC), U17.22 (NC)
- new net: Q1.1 (D), Q1.2 (D), Q1.5 (D), Q1.6 (D), Q1.8 (D)
- new net: Q1.4 (S), Q1.7 (S)
- new net 4.4V (ACTIONBUTTON LED RING): C8.2, J6.1 (Pin_1), P1.1, U11.1 (VCCA)
- new net 4.4V (LED STRIP 1 AND 2): C21.2, J1.1 (Pin_1), J2.1 (Pin_1), U14.1 (VCCA)
- new net 4.4V (LED STRIP 3 AND 4): C28.2, J3.1 (Pin_1), J4.1 (Pin_1), U24.1 (VCCA)
- new net DTR: U22.2 (B), U22.4 (E), U25.23 (DTR)
- new net ESP32 EN: C25.2, R22.2, SW4.2, U17.3 (EN)
- new net IO0: U22.3 (C)
- new net IO13/SPI MI: U17.16 (IO13)
- new net IO14/SPI MO: U17.13 (IO14)
- new net IO21/I2C SDA: U17.33 (IO21)
- new net IO22/I2C SCL: U17.36 (IO22)
- new net IO23/I2S WS: U10.2 (L/R), U17.37 (IO23)
- new net IO25/I2S SCK: U10.3 (CLK), U17.10 (IO25)
- new net IO26/I2S SD: U10.4 (DATA), U17.11 (IO26)
- new net IO27/ACTIONBUTTON LED RING: J6.2 (Pin_2), U11.7 (B1), U17.12 (IO27)
- new net IO32/ACTIONBUTTON: U15.4 (2Y), U17.8 (IO32)
- new net IO33/USB PD VOLTS DETECTION: U17.9 (IO33)
- new net IO4/SPI SCK: U17.26 (IO4)
- new net IO5/LED STRIPS POWER ON: U17.29 (IO5)
- new net RTS: U22.1 (E), U22.5 (B), U25.19 (RTS)
- new net USB-C D+: U2.6 (DP1), U2.8 (DP2), U25.3 (D+), U28.4
- new net USB-C D-: U2.5 (DN2), U2.7 (DN1), U25.4 (D-), U28.3
- no-connect marks 24 -> 31
Other:
- note added: "0A min"
- note added: "20V max"
- note added: "5V min"
- note added: "5V to 3.3V converter"
- note added: "8MB flash, 2MB PSRAM"
- note added: "Also make EN button accessible from the bottom of the LED lamp, without disassebling it first. For flashing, resetting and more."
- note added: "Auto program DTR RTS --> EN IO0 1 1 1 1 0 0 1 1 1 0 0 1 0 1 1 0"
- note added: "Autoreset"
- note added: "Fix MagiqWand and based on that see if microphone settings need to be updated in WLED."
- note added: "INFO: MOSFET has slightly different Vgs(th) values then recommended MOSFET. But should be fine. Original (BSL308PE H6327): -2.0 (min), -1.5 (typ), -1.0(max), condition ID=-11uA This model: -1.0 (min), -1.6 (typ), -3.0(max), condition ID=-250uA"
- note added: "Idea for turning CP2102N on/off: with mosfets like for GlowSign PCB (i think inspired by adafruit pcb design)"
- note added: "Many of the disconnected pins are required to be low or high on boot, or else prevent the ESP32 from booting. Therefore shouldn't be used."
- note added: "Need to test how to implement VBUS connection. Option 1: - voltage divider 20K and 5.1K resistors, connected to VBUS of USB C. - will result in output voltage on VBUS pin of 1V (if 5V power source) to 4V (if 20V USB PD source) Option 2: - connect directly to 3.3 output of buck/boost, which is powered by USB PD Test plan: - unsolder the existing voltage divider on the Adafruit CP2102N board - conn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"
- note added: "Protection diode can only handle 5V, so cannot be connected to VBUS (up to 20V). Option 1: - only connect to USB D+ and D- (and GND of course) Option 2: - connect also to 3.3V, if CP2102N will be powered directly via 3.3V pin"
- note added: "TODO: - can I test the behaviour at xhain with existing mosfets?"
- note added: "TODO: - request 9V 2A - add missing mosfets for safe_pwr?"
- note added: "TODO: - use MOSFETs to turn off/on the LED strips power (except for button LEDs, they always stay on)"
- note added: "TODOs: - Add switch to switch between GlowLight & GlowTower settings. - Make it accessible via backside - consider adding a resettable fuse"
- note added: "USB to Serial"
- note added: "USB-C PD (9-20V) to 5V"
- note added: "WARNING: I am not sure if the SAFE_5V_out is really designed for outputting 5V or only to send a signal. Falstadt says it stays at around 2.x v, not 5v. but then again... falstadt also says there will be 20v flowing throw it, if safe_pwr is off..."
- note added: "add capacitors?"
- note added: "connect remaining pin to have another external levelshifter connected led output onboard?"
- note added: "must be HIGH during boot, prevents startup log if pulled LOW"
- note added: "must be LOW during boot and also connected to the on-board LED"
- note added: "pin must be HIGH during boot"
- note added: "pin must be LOW during boot"
- note removed: "Designed for VIN 4.8V to 21V, at 1A max output. Based on webench.ti.com."
- note removed: "FINE SETTING +0"
- note removed: "GlowLight (2A)"
- note removed: "GlowLight (5V)"
- note removed: "GlowTower (20V)"
- note removed: "GlowTower (3A)"
- note removed: "ISNK_COARSE"
- note removed: "Status LED"
- note removed: "Stepdown converter will only turn on if USB_PD_IC_VDC_OUT is 9V or higher."
- note removed: "USB-C PD to 3.3V"
- note removed: "USB-C PD to 5V"
- note removed: "VBUS MAX 20V"
- note removed: "VBUS MIN"
- note removed: "VBUS to 5V"
- moved on the sheet: C14, C15, C19, C21, C23, C25, C28, C29, H2, R1, R24, R25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

Commit message: added more missing resistors for USB PD IC
Other:
- note added: "INFO: MOSFET has slightly different Vgs(th) values then recommended MOSFET. But should be fine. Original (BSL308PE H6327): -1.0 (min), -1.5 (typ), -2.0(max), condition ID=-11uA This model: -1.0 (min), -1.6 (typ), -3.0(max), condition ID=-250uA"
- note removed: "INFO: MOSFET has slightly different Vgs(th) values then recommended MOSFET. But should be fine. Original (BSL308PE H6327): -2.0 (min), -1.5 (typ), -1.0(max), condition ID=-11uA This model: -1.0 (min), -1.6 (typ), -3.0(max), condition ID=-250uA"
Changed lines of the file:
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@@
     (effects (font (size 1 1)) (justify left bottom))
   )
-  (text "INFO:\nMOSFET has slightly different Vgs(th) values then recommended MOSFET. But should be fine.\nOriginal (BSL308PE H6327):\n-2.0 (min), -1.5 (typ), -1.0(max), condition ID=-11uA\nThis model:\n-1.0 (min), -1.6 (typ), -3.0(max), condition ID=-250uA"
+  (text "INFO:\nMOSFET has slightly different Vgs(th) values then recommended MOSFET. But should be fine.\nOriginal (BSL308PE H6327):\n-1.0 (min), -1.5 (typ), -2.0(max), condition ID=-11uA\nThis model:\n-1.0 (min), -1.6 (typ), -3.0(max), condition ID=-250uA"
     (at 200.025 180.34 0)
     (effects (font (size 1 1)) (justify left bottom))
